File: v1/LoRaNow_v1.brd (EAGLE design)
At the start: 25.4 x 30.5 mm, 29 parts, among them Q1 MOSFET-PCHANNELSMD, Q2 8/16/20MHz, U1 ATMEGA328, U2 TPL5110

Commit message: Update
Parts:
- Q1: value MOSFET-PCHANNELSMD -> P-MOSFET
- RFM95: value LORANOW -> RFM95
Changed lines of the file:
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@@
 <drawing>
 <settings>
-<setting alwaysvectorfont="yes"/>
+<setting alwaysvectorfont="no"/>
 <setting verticaltext="up"/>
 </settings>
@@
 <attribute name="VALUE" x="10.16" y="27.178" size="0.6096" layer="27" font="vector" ratio="20"/>
 </element>
-<element name="Q1" library="User-Submitted" package="SOT23-3" value="MOSFET-PCHANNELSMD" x="13.335" y="23.97125" smashed="yes">
+<element name="Q1" library="User-Submitted" package="SOT23-3" value="P-MOSFET" x="13.335" y="23.97125" smashed="yes">
 <attribute name="NAME" x="13.30325" y="23.6855" size="0.6096" layer="25" font="vector" ratio="20" align="bottom-center"/>
 <attribute name="VALUE" x="12.319" y="23.78075" size="0.4064" layer="27"/>
@@
 <attribute name="VALUE" x="5.87375" y="13.04925" size="0.6096" layer="27" font="vector" ratio="20" align="top-center"/>
 </element>
-<element name="RFM95" library="diy-modules" package="WIRELESS-LORANOW-RFM95W#SMD#2" value="LORANOW" x="12.85875" y="16.1925" smashed="yes" rot="MR90">
+<element name="RFM95" library="diy-modules" package="WIRELESS-LORANOW-RFM95W#SMD#2" value="RFM95" x="12.85875" y="16.1925" smashed="yes" rot="MR90">
 <attribute name="NAME" x="17.30375" y="13.97" size="0.762" layer="26" font="vector" ratio="20" rot="MR90" align="center"/>
 <attribute name="VALUE" x="14.12875" y="13.97" size="0.762" layer="28" font="vector" ratio="20" rot="MR90" align="center"/>
