File: v1/LoRaNow_v1.sch (EAGLE design)
At the start: 27 parts, among them Q1 MOSFET-PCHANNELSMD, Q2 8/16/20MHz, U1 ATMEGA328, U2 TPL5110

Commit message: Update
Parts:
- Q1: value MOSFET-PCHANNELSMD -> P-MOSFET
- RFM95: value LORANOW -> RFM95
Changed lines of the file:
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@@
 <parts>
 <part name="J3" library="SparkFun-Connectors" deviceset="CONN_04" device="1X04_NO_SILK"/>
-<part name="Q1" library="User-Submitted" deviceset="MOSFET-PCHANNEL" device="SMD"/>
+<part name="Q1" library="User-Submitted" deviceset="MOSFET-PCHANNEL" device="SMD" value="P-MOSFET"/>
 <part name="R1" library="SparkFun-Resistors" deviceset="100KOHM" device="-0603-1/10W-1%" value="100k"/>
 <part name="ANTENNA" library="SparkFun-Connectors" deviceset="U.FL" device="U.FL_2A"/>
@@
 <part name="GND6" library="SparkFun" deviceset="GND" device=""/>
 <part name="P+3" library="SparkFun" deviceset="3.3V" device="" value="VCC"/>
-<part name="RFM95" library="diy-modules" deviceset="WIRELESS-LORANOW-RFM95W" device="WIRELESS-LORANOW-RFM95W#SMD#2" value="LORANOW"/>
+<part name="RFM95" library="diy-modules" deviceset="WIRELESS-LORANOW-RFM95W" device="WIRELESS-LORANOW-RFM95W#SMD#2" value="RFM95"/>
 <part name="GND7" library="SparkFun" deviceset="GND" device=""/>
 <part name="P+5" library="SparkFun" deviceset="3.3V" device="" value="VCC"/>
